Commit message: 更新天工3 URDF 至 V3

File: tiangong3_urdf/urdf/tiangong3.urdf (robot description, URDF)
Before this commit: robot tiangong3, 31 links, 30 joints
Links:
- added link elbow_yaw_l_link, mass 0.31993; collision mesh filename=package://tiangong3_0_V2_urdf/meshes/elbow_yaw_l_link.STL; visual mesh filename=package://tiangong3_0_V2_urdf/meshes/elbow_yaw_l_link.STL
- added link elbow_yaw_r_link, mass 0.31993; collision mesh filename=package://tiangong3_0_V2_urdf/meshes/elbow_yaw_r_link.STL; visual mesh filename=package://tiangong3_0_V2_urdf/meshes/elbow_yaw_r_link.STL
- added link left_tcp_link, mass 0.384094; collision mesh filename=package://tiangong3_0_V2_urdf/meshes/left_tcp_link.STL; visual mesh filename=package://tiangong3_0_V2_urdf/meshes/left_tcp_link.STL
- added link right_tcp_link, mass 0.384094; collision mesh filename=package://tiangong3_0_V2_urdf/meshes/right_tcp_link.STL; visual mesh filename=package://tiangong3_0_V2_urdf/meshes/right_tcp_link.STL
- added link wrist_pitch_l_link, mass 1.089228; collision mesh filename=package://tiangong3_0_V2_urdf/meshes/wrist_pitch_l_link.STL; visual mesh filename=package://tiangong3_0_V2_urdf/meshes/wrist_pitch_l_link.STL
- added link wrist_pitch_r_link, mass 1.089228; collision mesh filename=package://tiangong3_0_V2_urdf/meshes/wrist_pitch_r_link.STL; visual mesh filename=package://tiangong3_0_V2_urdf/meshes/wrist_pitch_r_link.STL
- added link wrist_roll_l_link, mass 0.162372; collision mesh filename=package://tiangong3_0_V2_urdf/meshes/wrist_roll_l_link.STL; visual mesh filename=package://tiangong3_0_V2_urdf/meshes/wrist_roll_l_link.STL
- added link wrist_roll_r_link, mass 0.162372; collision mesh filename=package://tiangong3_0_V2_urdf/meshes/wrist_roll_r_link.STL; visual mesh filename=package://tiangong3_0_V2_urdf/meshes/wrist_roll_r_link.STL
- link ankle_pitch_l_link: mass 0.142658 -> 0.122342; geometry collision mesh filename=package://tiangong3_0_V2_urdf/meshes/ankle_pitch_l_link.STL; visual mesh filename=package://tiangong3_0_V2_urdf/meshes/ankle_pitch_l_link.STL
- link ankle_pitch_r_link: mass 0.142658 -> 0.122342; geometry collision mesh filename=package://tiangong3_0_V2_urdf/meshes/ankle_pitch_r_link.STL; visual mesh filename=package://tiangong3_0_V2_urdf/meshes/ankle_pitch_r_link.STL
- link ankle_roll_l_link: mass 0.888892 -> 0.826437; geometry collision mesh filename=package://tiangong3_0_V2_urdf/meshes/ankle_roll_l_link.STL; visual mesh filename=package://tiangong3_0_V2_urdf/meshes/ankle_roll_l_link.STL
- link ankle_roll_r_link: mass 0.888892 -> 0.826437; geometry collision mesh filename=package://tiangong3_0_V2_urdf/meshes/ankle_roll_r_link.STL; visual mesh filename=package://tiangong3_0_V2_urdf/meshes/ankle_roll_r_link.STL
- link camera_body_front_link: geometry collision mesh filename=package://tiangong3_0_V2_urdf/meshes/camera_body_front_link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; visual mesh filename=package://tiangong3_0_V2_urdf/meshes/camera_body_front_link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
- link camera_head_link: geometry collision mesh filename=package://tiangong3_0_V2_urdf/meshes/camera_head_link.STL; visual mesh filename=package://tiangong3_0_V2_urdf/meshes/camera_head_link.STL
- link elbow_pitch_l_link: mass 0.531558 -> 0.762706; geometry collision mesh filename=package://tiangong3_0_V2_urdf/meshes/elbow_pitch_l_link.STL; visual mesh filename=package://tiangong3_0_V2_urdf/meshes/elbow_pitch_l_link.STL
- link elbow_pitch_r_link: mass 0.531558 -> 0.762706; geometry collision mesh filename=package://tiangong3_0_V2_urdf/meshes/elbow_pitch_r_link.STL; visual mesh filename=package://tiangong3_0_V2_urdf/meshes/elbow_pitch_r_link.STL
- link head_pitch_link: mass 0.087922 -> 0.077424; geometry collision mesh filename=package://tiangong3_0_V2_urdf/meshes/head_pitch_link.STL; visual mesh filename=package://tiangong3_0_V2_urdf/meshes/head_pitch_link.STL
- link head_yaw_link: mass 0.968233 -> 1.057204; geometry collision mesh filename=package://tiangong3_0_V2_urdf/meshes/head_yaw_link.STL; visual mesh filename=package://tiangong3_0_V2_urdf/meshes/head_yaw_link.STL
- link hip_pitch_l_link: mass 2.373121 -> 2.427595; geometry collision mesh filename=package://tiangong3_0_V2_urdf/meshes/hip_pitch_l_link.STL; visual mesh filename=package://tiangong3_0_V2_urdf/meshes/hip_pitch_l_link.STL
- link hip_pitch_r_link: mass 2.373121 -> 2.427595; geometry collision mesh filename=package://tiangong3_0_V2_urdf/meshes/hip_pitch_r_link.STL; visual mesh filename=package://tiangong3_0_V2_urdf/meshes/hip_pitch_r_link.STL
- link hip_roll_l_link: mass 0.539594 -> 0.578439; geometry collision mesh filename=package://tiangong3_0_V2_urdf/meshes/hip_roll_l_link.STL; visual mesh filename=package://tiangong3_0_V2_urdf/meshes/hip_roll_l_link.STL
- link hip_roll_r_link: mass 0.539594 -> 0.578439; geometry collision mesh filename=package://tiangong3_0_V2_urdf/meshes/hip_roll_r_link.STL; visual mesh filename=package://tiangong3_0_V2_urdf/meshes/hip_roll_r_link.STL
- link hip_yaw_l_link: mass 5.562147 -> 5.766953; geometry collision mesh filename=package://tiangong3_0_V2_urdf/meshes/hip_yaw_l_link.STL; visual mesh filename=package://tiangong3_0_V2_urdf/meshes/hip_yaw_l_link.STL
- link hip_yaw_r_link: mass 5.562147 -> 5.766953; geometry collision mesh filename=package://tiangong3_0_V2_urdf/meshes/hip_yaw_r_link.STL; visual mesh filename=package://tiangong3_0_V2_urdf/meshes/hip_yaw_r_link.STL
- link imu_head_link: geometry collision mesh filename=package://tiangong3_0_V2_urdf/meshes/imu_head_link.STL; visual mesh filename=package://tiangong3_0_V2_urdf/meshes/imu_head_link.STL
- link imu_waist_link: geometry collision mesh filename=package://tiangong3_0_V2_urdf/meshes/imu_waist_link.STL; visual mesh filename=package://tiangong3_0_V2_urdf/meshes/imu_waist_link.STL
- link knee_pitch_l_link: mass 2.945335 -> 3.14544; geometry collision mesh filename=package://tiangong3_0_V2_urdf/meshes/knee_pitch_l_link.STL; visual mesh filename=package://tiangong3_0_V2_urdf/meshes/knee_pitch_l_link.STL
- link knee_pitch_r_link: mass 2.945335 -> 3.14544; geometry collision mesh filename=package://tiangong3_0_V2_urdf/meshes/knee_pitch_r_link.STL; visual mesh filename=package://tiangong3_0_V2_urdf/meshes/knee_pitch_r_link.STL
- link pelvis: mass 11.528555 -> 11.09264; geometry collision mesh filename=package://tiangong3_0_V2_urdf/meshes/pelvis.STL; visual mesh filename=package://tiangong3_0_V2_urdf/meshes/pelvis.STL
- link radar_head_link: geometry collision mesh filename=package://tiangong3_0_V2_urdf/meshes/radar_head_link.STL; visual mesh filename=package://tiangong3_0_V2_urdf/meshes/radar_head_link.STL
- link shoulder_pitch_l_link: mass 0.914808 -> 0.967698; geometry collision mesh filename=package://tiangong3_0_V2_urdf/meshes/shoulder_pitch_l_link.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; visual mesh filename=package://tiangong3_0_V2_urdf/meshes/shoulder_pitch_l_link.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
- link shoulder_pitch_r_link: mass 0.914808 -> 0.967698; geometry collision mesh filename=package://tiangong3_0_V2_urdf/meshes/shoulder_pitch_r_link.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; visual mesh filename=package://tiangong3_0_V2_urdf/meshes/shoulder_pitch_r_link.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
- link shoulder_roll_l_link: mass 0.319153 -> 0.460858; geometry collision mesh filename=package://tiangong3_0_V2_urdf/meshes/shoulder_roll_l_link.S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; visual mesh filename=package://tiangong3_0_V2_urdf/meshes/shoulder_roll_l_link.S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
- link shoulder_roll_r_link: mass 0.319153 -> 0.460858; geometry collision mesh filename=package://tiangong3_0_V2_urdf/meshes/shoulder_roll_r_link.S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; visual mesh filename=package://tiangong3_0_V2_urdf/meshes/shoulder_roll_r_link.S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
- link shoulder_yaw_l_link: mass 1.502215 -> 1.53899; geometry collision mesh filename=package://tiangong3_0_V2_urdf/meshes/shoulder_yaw_l_link.STL; visual mesh filename=package://tiangong3_0_V2_urdf/meshes/shoulder_yaw_l_link.STL
- link shoulder_yaw_r_link: mass 1.502215 -> 1.53899; geometry collision mesh filename=package://tiangong3_0_V2_urdf/meshes/shoulder_yaw_r_link.STL; visual mesh filename=package://tiangong3_0_V2_urdf/meshes/shoulder_yaw_r_link.STL
- link waist_pitch_link: mass 10.400612 -> 9.973084; geometry collision mesh filename=package://tiangong3_0_V2_urdf/meshes/waist_pitch_link.STL; visual mesh filename=package://tiangong3_0_V2_urdf/meshes/waist_pitch_link.STL
- link waist_roll_link: mass 3.995987 -> 3.894484; geometry collision mesh filename=package://tiangong3_0_V2_urdf/meshes/waist_roll_link.STL; visual mesh filename=package://tiangong3_0_V2_urdf/meshes/waist_roll_link.STL
- link waist_yaw_link: mass 1.908803 -> 2.135803; geometry collision mesh filename=package://tiangong3_0_V2_urdf/meshes/waist_yaw_link.STL; visual mesh filename=package://tiangong3_0_V2_urdf/meshes/waist_yaw_link.STL
Joints:
- added joint elbow_yaw_l_joint: type revolute, parent elbow_pitch_l_link, child elbow_yaw_l_link, origin xyz=-0.02 0 -0.104 rpy=0 0 0, axis 0 0 1, limit lower=-2.844886680750757 upper=2.844886680750757 effort=40.0 velocity=18.325957145940457
- added joint elbow_yaw_r_joint: type revolute, parent elbow_pitch_r_link, child elbow_yaw_r_link, origin xyz=-0.02 0 -0.104 rpy=0 0 0, axis 0 0 1, limit lower=-2.844886680750757 upper=2.844886680750757 effort=40.0 velocity=18.325957145940457
- added joint left_tcp_joint: type fixed, parent wrist_roll_l_link, child left_tcp_link, origin xyz=0 0 -0.044 rpy=0 0 0, axis 0 0 0
- added joint right_tcp_joint: type fixed, parent wrist_roll_r_link, child right_tcp_link, origin xyz=0 0 -0.044 rpy=0 0 0, axis 0 0 0
- added joint wrist_pitch_l_joint: type revolute, parent elbow_yaw_l_link, child wrist_pitch_l_link, origin xyz=0 0 -0.0944 rpy=0 0 0, axis 0 1 0, limit lower=-1.3264502315156903 upper=1.3264502315156903 effort=40.0 velocity=18.325957145940457
- added joint wrist_pitch_r_joint: type revolute, parent elbow_yaw_r_link, child wrist_pitch_r_link, origin xyz=0 0 -0.0944 rpy=0 0 0, axis 0 1 0, limit lower=-1.3264502315156903 upper=1.3264502315156903 effort=40.0 velocity=18.325957145940457
- added joint wrist_roll_l_joint: type revolute, parent wrist_pitch_l_link, child wrist_roll_l_link, origin xyz=0 0 -0.062 rpy=0 0 0, axis 1 0 0, limit lower=-1.3264502315156903 upper=1.3264502315156903 effort=40.0 velocity=18.325957145940457
- added joint wrist_roll_r_joint: type revolute, parent wrist_pitch_r_link, child wrist_roll_r_link, origin xyz=0 0 -0.062 rpy=0 0 0, axis 1 0 0, limit lower=-1.3264502315156903 upper=1.3264502315156903 effort=40.0 velocity=18.325957145940457
- joint ankle_pitch_l_joint: origin xyz=0.0073681 0 -0.39993 rpy=0 0 0 -> xyz=0 0 -0.4 rpy=0 0 0
- joint ankle_pitch_r_joint: origin xyz=0.014553 0 -0.39974 rpy=0 0 0 -> xyz=0 0 -0.4 rpy=0 0 0
- joint knee_pitch_l_joint: origin xyz=-0.012927 0 -0.30599 rpy=0 0.018418 0 -> xyz=-0.012927 0 -0.30599 rpy=0 0 0
- joint knee_pitch_r_joint: origin xyz=-0.012927 0 -0.30599 rpy=0 0.036386 0 -> xyz=-0.012927 0 -0.30599 rpy=0 0 0
- joint waist_yaw_joint: limit lower=-2.6179938779914944 upper=3.2288591161895095 effort=91.0 velocity=9.42477796076938 -> lower=-2.6179938779914944 upper=3.2288591161895095 effort=200.0 velocity=10.053096491487338
