Commit message: 更新tianyi2.0带手的urdf文件

File: tianyi2_urdf/urdf/tianyi2.0_urdf_with_hands.urdf (robot description, URDF)
Before this commit: robot tianyi2.0_complete, 51 links, 50 joints
Joints:
- joint first_leg_pitch_joint: limit lower=-0.41887902047863906 upper=1.0471975511965976 effort=332.0 velocity=3.9269908169872414 -> lower=-0.41887902047863906 upper=0.9075712110370514 effort=332.0 velocity=3.9269908169872414
- joint second_leg_pitch_joint: limit lower=-0.5061454830783556 upper=1.7453292519943295 effort=332.0 velocity=3.9269908169872414 -> lower=-1.7453292519943295 upper=0.5061454830783556 effort=332.0 velocity=3.9269908169872414
- joint waist_pitch_joint: limit lower=-2.0943951023931953 upper=0.7853981633974483 effort=332.0 velocity=3.9269908169872414 -> lower=-0.7853981633974483 upper=2.0943951023931953 effort=332.0 velocity=3.9269908169872414
